File: MiSTer Vector v1.0.sch (EAGLE design)
At the start: 45 parts, among them CON2 22-23-2021, IC1 74HC00D, IC2 TL084, IC3 TL084, IC7 MAX6105, U1 MCP4922, U2 MCP4922, U3 MCP4922, U8 VASD1-SIP, X2 ILDA 25 Pin

Commit message: added VREF adj switch and pot, plus ILDA shutter jumper
Parts:
- added R14: (no value), pot:TRIM_EU-B25P
- added R15: 75R, resistor:R-US_R0603
- added SHUT: (no value), jumper:JP1E
- added XY_VREF_SW: (no value), adafruit:EG1218S
Connections:
- new net +VREF_XY: R5.1, R9.1, U1.REFA, U1.REFB, XY_VREF_SW.P
- new net N$12: R15.2, SHUT.1
- new net N$13: R14.S, XY_VREF_SW.S
- net +5V: now also R15.1
- net +VREF: now also R14.E, XY_VREF_SW.O; no longer R5.1, R9.1, U1.REFA, U1.REFB
- net GND: now also R14.A
- net SHUTTER: now also SHUT.2
Changed lines of the file:
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@@
 <part name="SUPPLY3" library="supply2" deviceset="GND" device=""/>
 <part name="D1" library="adafruit" deviceset="DIODE" device="SOD-323F"/>
+<part name="XY_VREF_SW" library="adafruit" deviceset="EG1218" device="S"/>
+<part name="R14" library="pot" deviceset="TRIM_EU-" device="B25P"/>
+<part name="SUPPLY19" library="supply2" deviceset="GND" device=""/>
+<part name="R15" library="resistor" deviceset="R-US_" device="R0603" value="75R"/>
+<part name="P+15" library="supply1" deviceset="+5V" device=""/>
+<part name="SHUT" library="jumper" deviceset="JP1E" device=""/>
 </parts>
 <sheets>
@@
 <instance part="SUPPLY3" gate="GND" x="-5.08" y="-5.08" rot="R270"/>
 <instance part="D1" gate="G$1" x="-17.78" y="-20.32"/>
+<instance part="XY_VREF_SW" gate="1" x="45.72" y="172.72" rot="MR270"/>
+<instance part="R14" gate="1" x="25.4" y="162.56"/>
+<instance part="SUPPLY19" gate="GND" x="25.4" y="152.4"/>
+<instance part="R15" gate="G$1" x="144.78" y="2.54"/>
+<instance part="P+15" gate="1" x="134.62" y="2.54" rot="MR270"/>
+<instance part="SHUT" gate="A" x="152.4" y="7.62"/>
 </instances>
 <busses>
@@
 <wire x1="0" y1="-5.08" x2="-2.54" y2="-5.08" width="0.1524" layer="91"/>
 </segment>
+<segment>
+<pinref part="SUPPLY19" gate="GND" pin="GND"/>
+<pinref part="R14" gate="1" pin="A"/>
+<wire x1="25.4" y1="154.94" x2="25.4" y2="157.48" width="0.1524" layer="91"/>
+</segment>
 </net>
 <net name="R+" class="0">
@@
 <wire x1="-40.64" y1="-20.32" x2="-35.56" y2="-20.32" width="0.1524" layer="91"/>
 </segment>
+<segment>
+<pinref part="P+15" gate="1" pin="+5V"/>
+<pinref part="R15" gate="G$1" pin="1"/>
+<wire x1="137.16" y1="2.54" x2="139.7" y2="2.54" width="0.1524" layer="91"/>
+</segment>
 </net>
 <net name="G1+" class="0">
@@
 </segment>
 <segment>
-<wire x1="78.74" y1="160.02" x2="71.12" y2="160.02" width="0.1524" layer="91"/>
-<label x="68.58" y="160.02" size="1.778" layer="95"/>
-<pinref part="R5" gate="G$1" pin="1"/>
-</segment>
-<segment>
-<wire x1="62.23" y1="125.73" x2="63.5" y2="125.73" width="0.1524" layer="91"/>
-<wire x1="63.5" y1="125.73" x2="63.5" y2="128.27" width="0.1524" layer="91"/>
-<wire x1="63.5" y1="128.27" x2="63.5" y2="130.81" width="0.1524" layer="91"/>
-<wire x1="63.5" y1="130.81" x2="62.23" y2="130.81" width="0.1524" layer="91"/>
-<wire x1="67.31" y1="128.27" x2="63.5" y2="128.27" width="0.1524" layer="91"/>
-<junction x="63.5" y="128.27"/>
-<label x="68.58" y="128.27" size="1.778" layer="95"/>
-<pinref part="U1" gate="U" pin="REFA"/>
-<pinref part="U1" gate="U" pin="REFB"/>
-</segment>
-<segment>
 <wire x1="62.23" y1="73.66" x2="63.5" y2="73.66" width="0.1524" layer="91"/>
 <wire x1="63.5" y1="73.66" x2="63.5" y2="71.12" width="0.1524" layer="91"/>
@@
 </segment>
 <segment>
-<pinref part="R9" gate="G$1" pin="1"/>
-<wire x1="78.74" y1="116.84" x2="73.66" y2="116.84" width="0.1524" layer="91"/>
-<label x="76.2" y="116.84" size="1.778" layer="95" rot="MR0"/>
+<pinref part="XY_VREF_SW" gate="1" pin="O"/>
+<pinref part="R14" gate="1" pin="E"/>
+<wire x1="40.64" y1="172.72" x2="25.4" y2="172.72" width="0.1524" layer="91"/>
+<wire x1="25.4" y1="172.72" x2="25.4" y2="167.64" width="0.1524" layer="91"/>
+<label x="30.48" y="172.72" size="1.778" layer="95"/>
 </segment>
 </net>
@@
 <pinref part="X2" gate="-1" pin="13"/>
 <label x="160.02" y="15.24" size="1.778" layer="95" rot="MR0"/>
+<wire x1="160.02" y1="2.54" x2="160.02" y2="15.24" width="0.1524" layer="91"/>
+<wire x1="160.02" y1="2.54" x2="154.94" y2="2.54" width="0.1524" layer="91"/>
+<pinref part="SHUT" gate="A" pin="2"/>
+<wire x1="154.94" y1="2.54" x2="154.94" y2="5.08" width="0.1524" layer="91"/>
 </segment>
 </net>
@@
 </segment>
 </net>
+<net name="+VREF_XY" class="0">
+<segment>
+<wire x1="62.23" y1="125.73" x2="63.5" y2="125.73" width="0.1524" layer="91"/>
+<wire x1="63.5" y1="125.73" x2="63.5" y2="128.27" width="0.1524" layer="91"/>
+<wire x1="63.5" y1="128.27" x2="63.5" y2="130.81" width="0.1524" layer="91"/>
+<wire x1="63.5" y1="130.81" x2="62.23" y2="130.81" width="0.1524" layer="91"/>
+<wire x1="67.31" y1="128.27" x2="63.5" y2="128.27" width="0.1524" layer="91"/>
+<junction x="63.5" y="128.27"/>
+<label x="68.58" y="128.27" size="1.778" layer="95"/>
+<pinref part="U1" gate="U" pin="REFA"/>
+<pinref part="U1" gate="U" pin="REFB"/>
+</segment>
+<segment>
+<pinref part="R9" gate="G$1" pin="1"/>
+<wire x1="78.74" y1="116.84" x2="73.66" y2="116.84" width="0.1524" layer="91"/>
+<label x="76.2" y="116.84" size="1.778" layer="95" rot="MR0"/>
+</segment>
+<segment>
+<wire x1="78.74" y1="160.02" x2="71.12" y2="160.02" width="0.1524" layer="91"/>
+<label x="68.58" y="160.02" size="1.778" layer="95"/>
+<pinref part="R5" gate="G$1" pin="1"/>
+</segment>
+<segment>
+<pinref part="XY_VREF_SW" gate="1" pin="P"/>
+<wire x1="50.8" y1="170.18" x2="55.88" y2="170.18" width="0.1524" layer="91"/>
+<label x="53.34" y="170.18" size="1.778" layer="95"/>
+</segment>
+</net>
+<net name="N$13" class="0">
+<segment>
+<pinref part="R14" gate="1" pin="S"/>
+<wire x1="30.48" y1="162.56" x2="35.56" y2="162.56" width="0.1524" layer="91"/>
+<wire x1="35.56" y1="162.56" x2="35.56" y2="167.64" width="0.1524" layer="91"/>
+<pinref part="XY_VREF_SW" gate="1" pin="S"/>
+<wire x1="35.56" y1="167.64" x2="40.64" y2="167.64" width="0.1524" layer="91"/>
+</segment>
+</net>
+<net name="N$12" class="0">
+<segment>
+<pinref part="SHUT" gate="A" pin="1"/>
+<pinref part="R15" gate="G$1" pin="2"/>
+<wire x1="152.4" y1="5.08" x2="152.4" y2="2.54" width="0.1524" layer="91"/>
+<wire x1="152.4" y1="2.54" x2="149.86" y2="2.54" width="0.1524" layer="91"/>
+</segment>
+</net>
